Commit message: Add files via upload

File: sizu_gazebo/urdf/robot.xacro (robot description, xacro)
@@ -2,7 +2,8 @@
     <xacro:include filename="sizu.urdf.xacro" />
     <xacro:include filename="sizu_transmission.xacro" />
+    <xacro:include filename="adhesion.xacro" />
     <gazebo>
         <plugin name="gazebo_ros_control" filename="libgazebo_ros_control.so">
-            <robotNamespace>/</robotNamespace>
+            <robotNamespace>/sizu</robotNamespace>
             <robotSimType>gazebo_ros_control/DefaultRobotHWSim</robotSimType>
         </plugin>
@@ -19,19 +20,19 @@
         </collision>
     </gazebo>
-    <gazebo reference="foot_FL">
-      <mu1>0.6</mu1>
-      <mu2>0.6</mu2>
+    <gazebo reference="tibia_FL">
+      <mu1>1</mu1>
+      <mu2>1</mu2>
     </gazebo>
-    <gazebo reference="foot_RL">
-      <mu1>0.6</mu1>
-      <mu2>0.6</mu2>
+    <gazebo reference="tibia_RL">
+      <mu1>1</mu1>
+      <mu2>1</mu2>
     </gazebo>
-    <gazebo reference="foot_FR">
-      <mu1>0.6</mu1>
-      <mu2>0.6</mu2>
+    <gazebo reference="tibia_FR">
+      <mu1>1</mu1>
+      <mu2>1</mu2>
     </gazebo>
-    <gazebo reference="foot_RR">
-      <mu1>0.6</mu1>
-      <mu2>0.6</mu2>
+    <gazebo reference="tibia_RR">
+      <mu1>1</mu1>
+      <mu2>1</mu2>
     </gazebo>
     <gazebo reference="lidar_link">
@@ -61,5 +62,5 @@
       </ray>
       <plugin name="gazebo_rplidar" filename="libgazebo_ros_laser.so">
-        <topicName>/scan</topicName>
+        <topicName>/sizu/scan</topicName>
         <frameName>lidar_link</frameName>
       </plugin>

File: sizu_gazebo/urdf/sizu.urdf.xacro (robot description, xacro)
@@ -19,17 +19,10 @@
   </joint>
   <!-- 机身 base_link -->
-  <link name="base_link">
+   <link name="base_link">
     <inertial>
       <origin xyz="0 0 0" rpy="0 0 0" />
       <mass value="3.0" />
-      <inertia
-        ixx="0.015"
-        ixy="0.0"
-        ixz="0.0"
-        iyy="0.020"
-        iyz="0.0"
-        izz="0.030" />
-    </inertial>
-    <!-- 高精度外观：保持 mesh 不变 -->
+      <inertia ixx="0.015" ixy="0.0" ixz="0.0" iyy="0.02" iyz="0.0" izz="0.03" />
+    </inertial>
     <visual>
       <origin xyz="0 0 0" rpy="0 0 0" />
@@ -38,16 +31,15 @@
       </geometry>
       <material name="">
-        <color rgba="1 1 1 1" />
-      </material>
-    </visual>
-    <!-- 简化碰撞：用机身实际尺寸的 box（长0.2305 宽0.2055 高0.05） -->
-    <collision>
-      <origin xyz="0 0 0" rpy="0 0 0" />
-      <geometry>
-        <box size="0.2305 0.2055 0.05"/>
-      </geometry>
-    </collision>
-  </link>
-  <link name="lidar_link">
+        <color rgba="1 1 1 0.5" />
+      </material>
+    </visual>
+    <collision>
+      <origin xyz="0 0 0" rpy="0 0 0" />
+      <geometry>
+        <box size="0.1705 0.1555 0.05"/>
+      </geometry>
+    </collision>
+  </link>
+ <link name="lidar_link">
     <visual>
       <origin xyz="0.01 0 -0.02" rpy="0 0 0" />
@@ -60,7 +52,7 @@
     </visual>
     <collision>
-      <origin xyz="0.1 0 0.08" rpy="0 0 0" />
-      <geometry>
-        <cylinder length="0.08" radius="0.04"/>
+      <origin xyz="0.01 0 -0.02" rpy="0 0 0" />
+      <geometry>
+        <cylinder length="0.04" radius="0.02"/>
       </geometry>
     </collision>
@@ -72,23 +64,14 @@
     <axis xyz="0 0 0" />
   </joint>
-  <!--=========================== FL 腿 ===========================-->
-  <link name="leg_center_FL">
-    <inertial>
-      <origin
-        xyz="-0.000984181618777502 -0.000539907314238933 -0.0344657673548433"
-        rpy="0 0 0" />
-      <mass value="0.151750032843904" />
-      <inertia
-        ixx="7.5000827940603E-05"
-        ixy="-1.80328417036782E-06"
-        ixz="1.62329378451308E-06"
-        iyy="7.72600969691206E-05"
-        iyz="8.8612311501709E-07"
-        izz="7.72691235265936E-05" />
-    </inertial>
-    <visual>
-      <origin xyz="0 0 0" rpy="0 0 0" />
-      <geometry>
-        <mesh filename="package://sizu_gazebo/meshes/leg_center_FL.STL" />
+  <link name="coxa_FL">
+    <inertial>
+      <origin xyz="0.04 0 0" rpy="0 0 0" />
+      <mass value="0.1" />
+      <inertia ixx="0.0001" ixy="0.0" ixz="0.0" iyy="0.0001" iyz="0.0" izz="0.0001" />
+    </inertial>
+    <visual>
+      <origin xyz="0 0 0" rpy="0 0 0" />
+      <geometry>
+        <mesh filename="package://sizu_gazebo/meshes/coxa_FL.STL" />
       </geometry>
       <material name="">
@@ -96,27 +79,107 @@
       </material>
     </visual>
-  </link>
-  <joint name="leg_center_joint_FL" type="fixed">
-    <origin xyz="0.164022451884239 0.128788837741078 0.0596" rpy="0 0 0" />
-    <parent link="base_link" />
-    <child link="leg_center_FL" />
-    <axis xyz="0 0 0" />
-  </joint>
-  <link name="coxa_FL">
-    <inertial>
-      <origin xyz="0 0 0" rpy="0 0 0" />
-      <mass value="0.0139" />
-      <inertia
-        ixx="2.0e-4"
-        ixy="0.0"
-        ixz="0.0"
-        iyy="3.0e-4"
-        iyz="0.0"
-        izz="3.0e-4" />
-    </inertial>
-    <visual>
-      <origin xyz="0 0 0" rpy="0 0 0" />
-      <geometry>
-        <mesh filename="package://sizu_gazebo/meshes/coxa_FL.STL" />
+    <collision>
+      <origin xyz="0.0 0 -0.02" rpy="0 0 0" />
+      <geometry>
+        <cylinder length="0.02" radius="0.02"/>
+      </geometry>
+    </collision>
+  </link>
+  <joint
+    name="coxa_joint_FL"
+    type="continuous">
+    <origin
+      xyz="0.10275 0.11525 0"
+      rpy="0 0 0" />
+    <parent
+      link="base_link" />
+    <child
+      link="coxa_FL" />
+    <axis
+      xyz="0 0 1" />
+    <limit effort="50" velocity="2"/>
+  </joint>
+  <link name="femur_FL">
+    <inertial>
+      <origin xyz="0.08 0 0" rpy="0 0 0" />
+      <mass value="0.5" />
+      <inertia ixx="0.003" ixy="0.0" ixz="0.0" iyy="0.003" iyz="0.0" izz="0.003" />
+    </inertial>
+    <visual>
+      <origin xyz="0 0 0" rpy="0 0 0" />
+      <geometry>
+        <mesh filename="package://sizu_gazebo/meshes/femur_FL.STL" />
+      </geometry>
+      <material name="">
+        <color rgba="0.8 0.8 0.8 1" />
+      </material>
+    </visual>
+    <collision>
+      <origin xyz="0.06 0 -0.02" rpy="0 0 0" />
+      <geometry>
+        <box size="0.12 0.04 0.04"/>
+      </geometry>
+    </collision>
+  </link>
+  <joint
+    name="femur_joint_FL"
+    type="continuous">
+    <origin
+      xyz="0.0635321928743235 0.0437332030011003 0.0255"
+      rpy="1.5707963267949 0 0.78539816339745" />
+    <parent
+      link="coxa_FL" />
+    <child
+      link="femur_FL" />
+    <axis
+      xyz="0 0 -1" />
+    <limit effort="50" velocity="2"/>
+  </joint>
+  <link name="tibia_FL">
+    <inertial>
+      <origin xyz="0.18 0 0" rpy="0 0 0" />
+      <mass value="0.2" />
+      <inertia ixx="0.002" ixy="0.0" ixz="0.0" iyy="0.002" iyz="0.0" izz="0.002" />
+    </inertial>
+    <visual>
+      <origin xyz="0 0 0" rpy="0 0 0" />
+      <geometry>
+        <mesh filename="package://sizu_gazebo/meshes/tibia_FL.STL" />
+      </geometry>
+      <material name="">
+        <color rgba="0.2 0.2 0.2 1" />
+      </material>
+    </visual>
+    <collision>
+      <origin xyz="0.18 0 0" rpy="0 0 0" />
+      <geometry>
+        <box size="0.26 0.03 0.03"/>
+      </geometry>
+    </collision>
+  </link>
+  <joint
+    name="tibia_joint_FL"
+    type="continuous">
+    <origin
+      xyz="0.164 0 0"
+      rpy="0 0 0" />
+    <parent
+      link="femur_FL" />
+    <child
+      link="tibia_FL" />
+    <axis
+      xyz="0 0 -1" />
+    <limit effort="50" velocity="2"/>
+  </joint>
+  <link name="coxa_RL">
+    <inertial>
+      <origin xyz="0.04 0 0" rpy="0 0 0" />
+      <mass value="0.1" />
+      <inertia ixx="0.0001" ixy="0.0" ixz="0.0" iyy="0.0001" iyz="0.0" izz="0.0001" />
+    </inertial>
+    <visual>
+      <origin xyz="0 0 0" rpy="0 0 0" />
+      <geometry>
+        <mesh filename="package://sizu_gazebo/meshes/coxa_RL.STL" />
       </geometry>
       <material name="">
@@ -124,35 +187,107 @@
       </material>
     </visual>
-    <!-- 简化碰撞：coxa 长 0.0633, 截面约 0.03x0.03 -->
-    <collision>
-      <origin xyz="0.03165 0 0" rpy="0 0 0" />
-      <geometry>
-        <box size="0.0633 0.03 0.03"/>
-      </geometry>
-    </collision>
-  </link>
-  <joint name="coxa_joint_FL" type="revolute">
-    <origin xyz="0 0 0" rpy="0 0 0.785" />
-    <parent link="leg_center_FL" />
-    <child link="coxa_FL" />
-    <axis xyz="0 0 1" />
-    <limit lower="-3.14" upper="3.14" effort="30" velocity="1" />
-  </joint>
-  <link name="femur_FL">
-    <inertial>
-      <origin xyz="0 0 0" rpy="0 0 0" />
-      <mass value="0.5649" />
-      <inertia
-        ixx="0.0030"
-        ixy="0.0"
-        ixz="0.0"
-        iyy="0.0015"
-        iyz="0.0"
-        izz="0.0040" />
-    </inertial>
-    <visual>
-      <origin xyz="0 0 0" rpy="0 0 0" />
-      <geometry>
-        <mesh filename="package://sizu_gazebo/meshes/femur_FL.STL" />
+    <collision>
+      <origin xyz="0.0 0 -0.02" rpy="0 0 0" />
+      <geometry>
+        <cylinder length="0.02" radius="0.02"/>
+      </geometry>
+    </collision>
+  </link>
+  <joint
+    name="coxa_joint_RL"
+    type="continuous">
+    <origin
+      xyz="-0.10275 0.11525 0"
+      rpy="0 0 0" />
+    <parent
+      link="base_link" />
+    <child
+      link="coxa_RL" />
+    <axis
+      xyz="0 0 1" />
+    <limit effort="50" velocity="2"/>
+  </joint>
+  <link name="femur_RL">
+    <inertial>
+      <origin xyz="0.08 0 0" rpy="0 0 0" />
+      <mass value="0.5" />
+      <inertia ixx="0.003" ixy="0.0" ixz="0.0" iyy="0.003" iyz="0.0" izz="0.003" />
+    </inertial>
+    <visual>
+      <origin xyz="0 0 0" rpy="0 0 0" />
+      <geometry>
+        <mesh filename="package://sizu_gazebo/meshes/femur_RL.STL" />
+      </geometry>
+      <material name="">
+        <color rgba="0.8 0.8 0.8 1" />
+      </material>
+    </visual>
+    <collision>
+      <origin xyz="0.06 0 -0.02" rpy="0 0 0" />
+      <geometry>
+        <box size="0.12 0.04 0.04"/>
+      </geometry>
+    </collision>
+  </link>
+  <joint
+    name="femur_joint_RL"
+    type="continuous">
+    <origin
+      xyz="-0.0635321928743236 0.0437332030011001 0.0255"
+      rpy="-1.5707963267949 0 2.35619449019235" />
+    <parent
+      link="coxa_RL" />
+    <child
+      link="femur_RL" />
+    <axis
+      xyz="0 0 -1" />
+    <limit effort="50" velocity="2"/>
+  </joint>
+  <link name="tibia_RL">
+    <inertial>
+      <origin xyz="0.18 0 0" rpy="0 0 0" />
+      <mass value="0.2" />
+      <inertia ixx="0.002" ixy="0.0" ixz="0.0" iyy="0.002" iyz="0.0" izz="0.002" />
+    </inertial>
+    <visual>
+      <origin xyz="0 0 0" rpy="0 0 0" />
+      <geometry>
+        <mesh filename="package://sizu_gazebo/meshes/tibia_RL.STL" />
+      </geometry>
+      <material name="">
+        <color rgba="0.2 0.2 0.2 1" />
+      </material>
+    </visual>
+    <collision>
+      <origin xyz="0.18 0 0" rpy="0 0 0" />
+      <geometry>
+        <box size="0.26 0.03 0.03"/>
+      </geometry>
+    </collision>
+  </link>
+  <joint
+    name="tibia_joint_RL"
+    type="continuous">
+    <origin
+      xyz="0.164 0 0"
+      rpy="0 0 0" />
+    <parent
+      link="femur_RL" />
+    <child
+      link="tibia_RL" />
+    <axis
+      xyz="0 0 -1" />
+    <limit effort="50" velocity="2"/>
+  </joint>
+  <link name="coxa_FR">
+    <inertial>
+      <origin xyz="0.04 0 0" rpy="0 0 0" />
+      <mass value="0.1" />
+      <inertia ixx="0.0001" ixy="0.0" ixz="0.0" iyy="0.0001" iyz="0.0" izz="0.0001" />
+    </inertial>
+    <visual>
+      <origin xyz="0 0 0" rpy="0 0 0" />
+      <geometry>
+        <mesh filename="package://sizu_gazebo/meshes/coxa_FR.STL" />
       </geometry>
       <material name="">
@@ -160,71 +295,107 @@
       </material>
     </visual>
-    <!-- 简化碰撞：femur 长 0.164, 主要沿 -Y 方向 -->
-    <collision>
-      <origin xyz="0 -0.1 -0.03" rpy="0 0 0" />
-      <geometry>
-        <box size="0.03 0.15 0.04"/>
-      </geometry>
-    </collision>
-  </link>
-  <joint name="femur_joint_FL" type="revolute">
-    <origin xyz="0.0718 0.0225 0.025" rpy="-1.57 1.56 0" />
-    <parent link="coxa_FL" />
-    <child link="femur_FL" />
-    <axis xyz="0 0 -1" />
-    <limit lower="-3.14" upper="3.14" effort="50" velocity="1" />
-  </joint>
-  <link name="tibia_FL">
-    <inertial>
-      <origin xyz="0 0 0" rpy="0 0 0" />
-      <mass value="0.2240" />
-      <inertia
-        ixx="0.0020"
-        ixy="0.0"
-        ixz="0.0"
-        iyy="0.0008"
-        iyz="0.0"
-        izz="0.0025" />
-    </inertial>
-    <visual>
-      <origin xyz="0 0 0" rpy="0 0 0" />
-      <geometry>
-        <mesh filename="package://sizu_gazebo/meshes/tibia_FL.STL" />
-      </geometry>
-      <material name="">
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