Commit message: Add files via upload

File: sizu_gazebo/urdf/robot.xacro (robot description, xacro)
@@ -2,5 +2,4 @@
     <xacro:include filename="sizu.urdf.xacro" />
     <xacro:include filename="sizu_transmission.xacro" />
-    <xacro:include filename="adhesion.xacro" />
     <gazebo>
         <plugin name="gazebo_ros_control" filename="libgazebo_ros_control.so">
@@ -8,5 +7,5 @@
             <robotSimType>gazebo_ros_control/DefaultRobotHWSim</robotSimType>
         </plugin>
-        <plugin name="collision_visualizer" filename="libcollision_map_creator.so"/>
+        <!-- <plugin name="collision_visualizer" filename="libcollision_map_creator.so"/> -->
         <!-- Gazebo专用标签 -->
         <collision>
@@ -19,20 +18,4 @@
          </surface>
         </collision>
-    </gazebo>
-    <gazebo reference="tibia_FL">
-      <mu1>1</mu1>
-      <mu2>1</mu2>
-    </gazebo>
-    <gazebo reference="tibia_RL">
-      <mu1>1</mu1>
-      <mu2>1</mu2>
-    </gazebo>
-    <gazebo reference="tibia_FR">
-      <mu1>1</mu1>
-      <mu2>1</mu2>
-    </gazebo>
-    <gazebo reference="tibia_RR">
-      <mu1>1</mu1>
-      <mu2>1</mu2>
     </gazebo>
     <gazebo reference="lidar_link">
@@ -67,3 +50,27 @@
     </sensor>
   </gazebo>
+  <gazebo>
+    <plugin filename="libgazebo_ros_force.so" name="gazebo_ros_force_tibia_FL">
+      <bodyName>tibia_FL</bodyName>
+      <topicName>/apply_force/tibia_FL</topicName>
+    </plugin>
+  </gazebo>
+  <gazebo>
+    <plugin filename="libgazebo_ros_force.so" name="gazebo_ros_force_tibia_FR">
+      <bodyName>tibia_FR</bodyName>
+      <topicName>/apply_force/tibia_FR</topicName>
+    </plugin>
+  </gazebo>
+  <gazebo>
+    <plugin filename="libgazebo_ros_force.so" name="gazebo_ros_force_tibia_RL">
+      <bodyName>tibia_RL</bodyName>
+      <topicName>/apply_force/tibia_RL</topicName>
+    </plugin>
+  </gazebo>
+  <gazebo>
+    <plugin filename="libgazebo_ros_force.so" name="gazebo_ros_force_tibia_RR">
+      <bodyName>tibia_RR</bodyName>
+      <topicName>/apply_force/tibia_RR</topicName>
+    </plugin>
+  </gazebo>
 </robot>

File: sizu_gazebo/urdf/sizu.urdf.xacro (robot description, xacro)
@@ -22,6 +22,6 @@
     <inertial>
       <origin xyz="0 0 0" rpy="0 0 0" />
-      <mass value="3.0" />
-      <inertia ixx="0.015" ixy="0.0" ixz="0.0" iyy="0.02" iyz="0.0" izz="0.03" />
+      <mass value="3.2" />
+      <inertia ixx="0.0085" ixy="0.0" ixz="0.0" iyy="0.0095" iyz="0.0" izz="0.0140" />
     </inertial>
     <visual>
@@ -41,9 +41,75 @@
     </collision>
   </link>
- <link name="lidar_link">
-    <visual>
-      <origin xyz="0.01 0 -0.02" rpy="0 0 0" />
-      <geometry>
-        <cylinder length="0.04" radius="0.02"/>
+  <!-- ==================== FL Leg ==================== -->
+  <link name="coxa_FL">
+    <inertial>
+      <origin xyz="0.04 0 0" rpy="0 0 0" />
+      <mass value="0.08" />
+      <inertia ixx="1.5e-5" ixy="0.0" ixz="0.0" iyy="5.0e-5" iyz="0.0" izz="5.0e-5" />
+    </inertial>
+    <visual>
+      <origin xyz="0 0 0" rpy="0 0 0" />
+      <geometry>
+        <mesh filename="package://sizu_gazebo/meshes/coxa_FL.STL" />
+      </geometry>
+      <material name="">
+        <color rgba="1 1 1 1" />
+      </material>
+    </visual>
+    <collision>
+      <origin xyz="0.0 0 -0.02" rpy="0 0 0" />
+      <geometry>
+        <cylinder length="0.02" radius="0.02"/>
+      </geometry>
+    </collision>
+  </link>
+  <joint name="coxa_joint_FL" type="revolute">
+    <origin xyz="0.10275 0.11525 0" rpy="0 0 0" />
+    <parent link="base_link" />
+    <child link="coxa_FL" />
+    <axis xyz="0 0 1" />
+    <dynamics damping="0.2" friction="0.02" />
+    <limit lower="-0.9" upper="0.9" effort="60" velocity="12"/>
+  </joint>
+  <link name="femur_FL">
+    <inertial>
+      <origin xyz="0.08 0 0" rpy="0 0 0" />
+      <mass value="0.32" />
+      <inertia ixx="8.0e-5" ixy="0.0" ixz="0.0" iyy="7.5e-4" iyz="0.0" izz="7.5e-4" />
+    </inertial>
+    <visual>
+      <origin xyz="0 0 0" rpy="0 0 0" />
+      <geometry>
+        <mesh filename="package://sizu_gazebo/meshes/femur_FL.STL" />
+      </geometry>
+      <material name="">
+        <color rgba="0.8 0.8 0.8 1" />
+      </material>
+    </visual>
+    <collision>
+      <origin xyz="0.08 0 -0.015" rpy="0 0 0" />
+      <geometry>
+        <box size="0.14 0.03 0.03"/>
+      </geometry>
+    </collision>
+  </link>
+  <joint name="femur_joint_FL" type="revolute">
+    <origin xyz="0.0635321928743235 0.0437332030011003 0.0255" rpy="1.5707963267949 0 0.78539816339745" />
+    <parent link="coxa_FL" />
+    <child link="femur_FL" />
+    <axis xyz="0 0 -1" />
+    <dynamics damping="0.2" friction="0.02" />
+    <limit lower="-1.6" upper="1.6" effort="60" velocity="16"/>
+  </joint>
+  <link name="tibia_FL">
+    <inertial>
+      <origin xyz="0.16 0 0" rpy="0 0 0" />
+      <mass value="0.16" />
+      <inertia ixx="2.0e-5" ixy="0.0" ixz="0.0" iyy="8.0e-4" iyz="0.0" izz="8.0e-4" />
+    </inertial>
+    <visual>
+      <origin xyz="0 0 0" rpy="0 0 0" />
+      <geometry>
+        <mesh filename="package://sizu_gazebo/meshes/tibia_FL.STL" />
       </geometry>
       <material name="">
@@ -52,26 +118,174 @@
     </visual>
     <collision>
-      <origin xyz="0.01 0 -0.02" rpy="0 0 0" />
-      <geometry>
-        <cylinder length="0.04" radius="0.02"/>
-      </geometry>
-    </collision>
-  </link>
-  <joint name="lidar_joint" type="fixed">
-    <origin xyz="0.1 0 0.08" rpy="0 0 0" />
+      <origin xyz="0.16 0 0" rpy="0 0 0" />
+      <geometry>
+        <box size="0.22 0.022 0.022"/>
+      </geometry>
+    </collision>
+  </link>
+  <joint name="tibia_joint_FL" type="revolute">
+    <origin xyz="0.164 0 0" rpy="0 0 0" />
+    <parent link="femur_FL" />
+    <child link="tibia_FL" />
+    <axis xyz="0 0 -1" />
+    <dynamics damping="0.2" friction="0.02" />
+    <limit lower="-2.4" upper="2.4" effort="60" velocity="16"/>
+  </joint>
+  <joint name="foot_fixed_FL" type="fixed" dont_collapse="true">
+    <origin xyz="0.31 0 0" rpy="0 0 0" />
+    <parent link="tibia_FL" />
+    <child link="foot_FL" />
+  </joint>
+  <link name="foot_FL">
+    <inertial>
+      <origin xyz="0 0 0" rpy="0 0 0" />
+      <mass value="0.03" />
+      <inertia ixx="4.0e-6" ixy="0.0" ixz="0.0" iyy="4.0e-6" iyz="0.0" izz="4.0e-6" />
+    </inertial>
+    <visual>
+      <origin xyz="0 0 0" rpy="0 0 0" />
+      <geometry>
+        <sphere radius="0.01"/>
+      </geometry>
+      <material name="">
+        <color rgba="0.1 0.1 0.1 1" />
+      </material>
+    </visual>
+    <collision>
+      <origin xyz="0 0 0" rpy="0 0 0" />
+      <geometry>
+        <sphere radius="0.016"/>
+      </geometry>
+    </collision>
+  </link>
+  <!-- ==================== RL Leg ==================== -->
+  <link name="coxa_RL">
+    <inertial>
+      <origin xyz="0.04 0 0" rpy="0 0 0" />
+      <mass value="0.08" />
+      <inertia ixx="1.5e-5" ixy="0.0" ixz="0.0" iyy="5.0e-5" iyz="0.0" izz="5.0e-5" />
+    </inertial>
+    <visual>
+      <origin xyz="0 0 0" rpy="0 0 0" />
+      <geometry>
+        <mesh filename="package://sizu_gazebo/meshes/coxa_RL.STL" />
+      </geometry>
+      <material name="">
+        <color rgba="1 1 1 1" />
+      </material>
+    </visual>
+    <collision>
+      <origin xyz="0.0 0 -0.02" rpy="0 0 0" />
+      <geometry>
+        <cylinder length="0.02" radius="0.02"/>
+      </geometry>
+    </collision>
+  </link>
+  <joint name="coxa_joint_RL" type="revolute">
+    <origin xyz="-0.10275 0.11525 0" rpy="0 0 0" />
     <parent link="base_link" />
-    <child link="lidar_link" />
-    <axis xyz="0 0 0" />
-  </joint>
-  <link name="coxa_FL">
+    <child link="coxa_RL" />
+    <axis xyz="0 0 1" />
+    <dynamics damping="0.2" friction="0.02" />
+    <limit lower="-0.9" upper="0.9" effort="60" velocity="12"/>
+  </joint>
+  <link name="femur_RL">
+    <inertial>
+      <origin xyz="0.08 0 0" rpy="0 0 0" />
+      <mass value="0.32" />
+      <inertia ixx="8.0e-5" ixy="0.0" ixz="0.0" iyy="7.5e-4" iyz="0.0" izz="7.5e-4" />
+    </inertial>
+    <visual>
+      <origin xyz="0 0 0" rpy="0 0 0" />
+      <geometry>
+        <mesh filename="package://sizu_gazebo/meshes/femur_RL.STL" />
+      </geometry>
+      <material name="">
+        <color rgba="0.8 0.8 0.8 1" />
+      </material>
+    </visual>
+    <collision>
+      <origin xyz="0.08 0 -0.015" rpy="0 0 0" />
+      <geometry>
+        <box size="0.14 0.03 0.03"/>
+      </geometry>
+    </collision>
+  </link>
+  <joint name="femur_joint_RL" type="revolute">
+    <origin xyz="-0.0635321928743236 0.0437332030011001 0.0255" rpy="-1.5707963267949 0 2.35619449019235" />
+    <parent link="coxa_RL" />
+    <child link="femur_RL" />
+    <axis xyz="0 0 -1" />
+    <dynamics damping="0.2" friction="0.02" />
+    <limit lower="-1.6" upper="1.6" effort="60" velocity="16"/>
+  </joint>
+  <link name="tibia_RL">
+    <inertial>
+      <origin xyz="0.16 0 0" rpy="0 0 0" />
+      <mass value="0.16" />
+      <inertia ixx="2.0e-5" ixy="0.0" ixz="0.0" iyy="8.0e-4" iyz="0.0" izz="8.0e-4" />
+    </inertial>
+    <visual>
+      <origin xyz="0 0 0" rpy="0 0 0" />
+      <geometry>
+        <mesh filename="package://sizu_gazebo/meshes/tibia_RL.STL" />
+      </geometry>
+      <material name="">
+        <color rgba="0.2 0.2 0.2 1" />
+      </material>
+    </visual>
+    <collision>
+      <origin xyz="0.16 0 0" rpy="0 0 0" />
+      <geometry>
+        <box size="0.22 0.022 0.022"/>
+      </geometry>
+    </collision>
+  </link>
+  <joint name="tibia_joint_RL" type="revolute">
+    <origin xyz="0.164 0 0" rpy="0 0 0" />
+    <parent link="femur_RL" />
+    <child link="tibia_RL" />
+    <axis xyz="0 0 -1" />
+    <dynamics damping="0.2" friction="0.02" />
+    <limit lower="-2.4" upper="2.4" effort="60" velocity="16"/>
+  </joint>
+  <joint name="foot_fixed_RL" type="fixed" dont_collapse="true">
+    <origin xyz="0.31 0 0" rpy="0 0 0" />
+    <parent link="tibia_RL" />
+    <child link="foot_RL" />
+  </joint>
+  <link name="foot_RL">
+    <inertial>
+      <origin xyz="0 0 0" rpy="0 0 0" />
+      <mass value="0.03" />
+      <inertia ixx="4.0e-6" ixy="0.0" ixz="0.0" iyy="4.0e-6" iyz="0.0" izz="4.0e-6" />
+    </inertial>
+    <visual>
+      <origin xyz="0 0 0" rpy="0 0 0" />
+      <geometry>
+        <sphere radius="0.01"/>
+      </geometry>
+      <material name="">
+        <color rgba="0.1 0.1 0.1 1" />
+      </material>
+    </visual>
+    <collision>
+      <origin xyz="0 0 0" rpy="0 0 0" />
+      <geometry>
+        <sphere radius="0.016"/>
+      </geometry>
+    </collision>
+  </link>
+  <!-- ==================== FR Leg ==================== -->
+  <link name="coxa_FR">
     <inertial>
       <origin xyz="0.04 0 0" rpy="0 0 0" />
-      <mass value="0.1" />
-      <inertia ixx="0.0001" ixy="0.0" ixz="0.0" iyy="0.0001" iyz="0.0" izz="0.0001" />
-    </inertial>
-    <visual>
-      <origin xyz="0 0 0" rpy="0 0 0" />
-      <geometry>
-        <mesh filename="package://sizu_gazebo/meshes/coxa_FL.STL" />
+      <mass value="0.08" />
+      <inertia ixx="1.5e-5" ixy="0.0" ixz="0.0" iyy="5.0e-5" iyz="0.0" izz="5.0e-5" />
+    </inertial>
+    <visual>
+      <origin xyz="0 0 0" rpy="0 0 0" />
+      <geometry>
+        <mesh filename="package://sizu_gazebo/meshes/coxa_FR.STL" />
       </geometry>
       <material name="">
@@ -86,28 +300,22 @@
     </collision>
   </link>
-  <joint
-    name="coxa_joint_FL"
-    type="continuous">
-    <origin
-      xyz="0.10275 0.11525 0"
-      rpy="0 0 0" />
-    <parent
-      link="base_link" />
-    <child
-      link="coxa_FL" />
-    <axis
-      xyz="0 0 1" />
-    <limit effort="50" velocity="2"/>
-  </joint>
-  <link name="femur_FL">
+  <joint name="coxa_joint_FR" type="revolute">
+    <origin xyz="0.10275 -0.11525 0" rpy="0 0 0" />
+    <parent link="base_link" />
+    <child link="coxa_FR" />
+    <axis xyz="0 0 1" />
+    <dynamics damping="0.2" friction="0.02" />
+    <limit lower="-0.9" upper="0.9" effort="60" velocity="12"/>
+  </joint>
+  <link name="femur_FR">
     <inertial>
       <origin xyz="0.08 0 0" rpy="0 0 0" />
-      <mass value="0.5" />
-      <inertia ixx="0.003" ixy="0.0" ixz="0.0" iyy="0.003" iyz="0.0" izz="0.003" />
-    </inertial>
-    <visual>
-      <origin xyz="0 0 0" rpy="0 0 0" />
-      <geometry>
-        <mesh filename="package://sizu_gazebo/meshes/femur_FL.STL" />
+      <mass value="0.32" />
+      <inertia ixx="8.0e-5" ixy="0.0" ixz="0.0" iyy="7.5e-4" iyz="0.0" izz="7.5e-4" />
+    </inertial>
+    <visual>
+      <origin xyz="0 0 0" rpy="0 0 0" />
+      <geometry>
+        <mesh filename="package://sizu_gazebo/meshes/femur_FR.STL" />
       </geometry>
       <material name="">
@@ -116,34 +324,28 @@
     </visual>
     <collision>
-      <origin xyz="0.06 0 -0.02" rpy="0 0 0" />
-      <geometry>
-        <box size="0.12 0.04 0.04"/>
-      </geometry>
-    </collision>
-  </link>
-  <joint
-    name="femur_joint_FL"
-    type="continuous">
-    <origin
-      xyz="0.0635321928743235 0.0437332030011003 0.0255"
-      rpy="1.5707963267949 0 0.78539816339745" />
-    <parent
-      link="coxa_FL" />
-    <child
-      link="femur_FL" />
-    <axis
-      xyz="0 0 -1" />
-    <limit effort="50" velocity="2"/>
-  </joint>
-  <link name="tibia_FL">
-    <inertial>
-      <origin xyz="0.18 0 0" rpy="0 0 0" />
-      <mass value="0.2" />
-      <inertia ixx="0.002" ixy="0.0" ixz="0.0" iyy="0.002" iyz="0.0" izz="0.002" />
-    </inertial>
-    <visual>
-      <origin xyz="0 0 0" rpy="0 0 0" />
-      <geometry>
-        <mesh filename="package://sizu_gazebo/meshes/tibia_FL.STL" />
+      <origin xyz="0.08 0 -0.015" rpy="0 0 0" />
+      <geometry>
+        <box size="0.14 0.03 0.03"/>
+      </geometry>
+    </collision>
+  </link>
+  <joint name="femur_joint_FR" type="revolute">
+    <origin xyz="0.0635321928743236 -0.0437332030011001 0.0255000000000001" rpy="-1.5707963267949 0 -0.785398163397447" />
+    <parent link="coxa_FR" />
+    <child link="femur_FR" />
+    <axis xyz="0 0 -1" />
+    <dynamics damping="0.2" friction="0.02" />
+    <limit lower="-1.6" upper="1.6" effort="60" velocity="16"/>
+  </joint>
+  <link name="tibia_FR">
+    <inertial>
+      <origin xyz="0.16 0 0" rpy="0 0 0" />
+      <mass value="0.16" />
+      <inertia ixx="2.0e-5" ixy="0.0" ixz="0.0" iyy="8.0e-4" iyz="0.0" izz="8.0e-4" />
+    </inertial>
+    <visual>
+      <origin xyz="0 0 0" rpy="0 0 0" />
+      <geometry>
+        <mesh filename="package://sizu_gazebo/meshes/tibia_FR.STL" />
       </geometry>
       <material name="">
@@ -152,34 +354,56 @@
     </visual>
     <collision>
-      <origin xyz="0.18 0 0" rpy="0 0 0" />
-      <geometry>
-        <box size="0.26 0.03 0.03"/>
-      </geometry>
-    </collision>
-  </link>
-  <joint
-    name="tibia_joint_FL"
-    type="continuous">
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