Commit message: Add files via upload

File: sizu_gazebo/urdf/robot.xacro (robot description, xacro)
@@ -50,3 +50,27 @@
     </sensor>
   </gazebo>
+  <gazebo>
+    <plugin filename="libgazebo_ros_force.so" name="gazebo_ros_force_tibia_FL">
+      <bodyName>tibia_FL</bodyName>
+      <topicName>/apply_force/tibia_FL</topicName>
+    </plugin>
+  </gazebo>
+  <gazebo>
+    <plugin filename="libgazebo_ros_force.so" name="gazebo_ros_force_tibia_FR">
+      <bodyName>tibia_FR</bodyName>
+      <topicName>/apply_force/tibia_FR</topicName>
+    </plugin>
+  </gazebo>
+  <gazebo>
+    <plugin filename="libgazebo_ros_force.so" name="gazebo_ros_force_tibia_RL">
+      <bodyName>tibia_RL</bodyName>
+      <topicName>/apply_force/tibia_RL</topicName>
+    </plugin>
+  </gazebo>
+  <gazebo>
+    <plugin filename="libgazebo_ros_force.so" name="gazebo_ros_force_tibia_RR">
+      <bodyName>tibia_RR</bodyName>
+      <topicName>/apply_force/tibia_RR</topicName>
+    </plugin>
+  </gazebo>
 </robot>

File: sizu_gazebo/urdf/sizu.urdf.xacro (robot description, xacro)
@@ -4,5 +4,6 @@
      For more information, please see http://wiki.ros.org/sw_urdf_exporter -->
 <robot xmlns:xacro="http://ros.org/wiki/xacro" name="sizu">
- <link name="map">
+  <!-- 过渡用 base（很小的可视box，不参与物理） -->
+  <link name="map">
     <visual>
       <origin xyz="0.0 0.0 0.0" rpy="0.0 0.0 0.0" />
@@ -21,6 +22,6 @@
     <inertial>
       <origin xyz="0 0 0" rpy="0 0 0" />
-      <mass value="3.2" />
-      <inertia ixx="0.0085" ixy="0.0" ixz="0.0" iyy="0.0095" iyz="0.0" izz="0.0140" />
+      <mass value="5.0" />
+      <inertia ixx="0.015" ixy="0.0" ixz="0.0" iyy="0.02" iyz="0.0" izz="0.03" />
     </inertial>
     <visual>
@@ -40,26 +41,32 @@
     </collision>
   </link>
-  <link name="lidar_link">
-    <visual>
-      <origin xyz="0 0 0" rpy="0 0 0" />
-      <geometry>
-        <cylinder radius="0.015" length="0.03"/>
-      </geometry>
-      <material name="black">
-        <color rgba="0.1 0.1 0.1 1.0" />
-      </material>
-    </visual>
+ <link name="lidar_link">
+    <visual>
+      <origin xyz="0.01 0 -0.02" rpy="0 0 0" />
+      <geometry>
+        <cylinder length="0.04" radius="0.02"/>
+      </geometry>
+      <material name="">
+        <color rgba="0.2 0.2 0.2 1" />
+      </material>
+    </visual>
+    <collision>
+      <origin xyz="0.01 0 -0.02" rpy="0 0 0" />
+      <geometry>
+        <cylinder length="0.04" radius="0.02"/>
+      </geometry>
+    </collision>
   </link>
   <joint name="lidar_joint" type="fixed">
-    <parent link="base_link"/>
-    <child link="lidar_link"/>
-    <origin xyz="0.0 0.0 0.08" rpy="0 0 0"/>
-  </joint>
-  <!-- ==================== FL Leg ==================== -->
+    <origin xyz="0.1 0 0.08" rpy="0 0 0" />
+    <parent link="base_link" />
+    <child link="lidar_link" />
+    <axis xyz="0 0 0" />
+  </joint>
   <link name="coxa_FL">
     <inertial>
       <origin xyz="0.04 0 0" rpy="0 0 0" />
-      <mass value="0.08" />
-      <inertia ixx="1.5e-5" ixy="0.0" ixz="0.0" iyy="5.0e-5" iyz="0.0" izz="5.0e-5" />
+      <mass value="0.15" />
+      <inertia ixx="0.0001" ixy="0.0" ixz="0.0" iyy="0.0001" iyz="0.0" izz="0.0001" />
     </inertial>
     <visual>
@@ -79,17 +86,23 @@
     </collision>
   </link>
-  <joint name="coxa_joint_FL" type="revolute">
-    <origin xyz="0.10275 0.11525 0" rpy="0 0 0" />
-    <parent link="base_link" />
-    <child link="coxa_FL" />
-    <axis xyz="0 0 1" />
-    <dynamics damping="0.2" friction="0.02" />
-    <limit lower="-0.9" upper="0.9" effort="60" velocity="12"/>
+  <joint
+    name="coxa_joint_FL"
+    type="continuous">
+    <origin
+      xyz="0.10275 0.11525 0"
+      rpy="0 0 0" />
+    <parent
+      link="base_link" />
+    <child
+      link="coxa_FL" />
+    <axis
+      xyz="0 0 1" />
+    <limit effort="50" velocity="2"/>
   </joint>
   <link name="femur_FL">
     <inertial>
       <origin xyz="0.08 0 0" rpy="0 0 0" />
-      <mass value="0.32" />
-      <inertia ixx="8.0e-5" ixy="0.0" ixz="0.0" iyy="7.5e-4" iyz="0.0" izz="7.5e-4" />
+      <mass value="1.5" />
+      <inertia ixx="0.003" ixy="0.0" ixz="0.0" iyy="0.003" iyz="0.0" izz="0.003" />
     </inertial>
     <visual>
@@ -103,23 +116,29 @@
     </visual>
     <collision>
-      <origin xyz="0.08 0 -0.015" rpy="0 0 0" />
-      <geometry>
-        <box size="0.14 0.03 0.03"/>
-      </geometry>
-    </collision>
-  </link>
-  <joint name="femur_joint_FL" type="revolute">
-    <origin xyz="0.0635321928743235 0.0437332030011003 0.0255" rpy="1.5707963267949 0 0.78539816339745" />
-    <parent link="coxa_FL" />
-    <child link="femur_FL" />
-    <axis xyz="0 0 -1" />
-    <dynamics damping="0.2" friction="0.02" />
-    <limit lower="-1.6" upper="1.6" effort="60" velocity="16"/>
+      <origin xyz="0.06 0 -0.02" rpy="0 0 0" />
+      <geometry>
+        <box size="0.12 0.04 0.04"/>
+      </geometry>
+    </collision>
+  </link>
+  <joint
+    name="femur_joint_FL"
+    type="continuous">
+    <origin
+      xyz="0.0635321928743235 0.0437332030011003 0.0255"
+      rpy="1.5707963267949 0 0.78539816339745" />
+    <parent
+      link="coxa_FL" />
+    <child
+      link="femur_FL" />
+    <axis
+      xyz="0 0 -1" />
+    <limit effort="50" velocity="2"/>
   </joint>
   <link name="tibia_FL">
     <inertial>
-      <origin xyz="0.16 0 0" rpy="0 0 0" />
-      <mass value="0.16" />
-      <inertia ixx="2.0e-5" ixy="0.0" ixz="0.0" iyy="8.0e-4" iyz="0.0" izz="8.0e-4" />
+      <origin xyz="0.18 0 0" rpy="0 0 0" />
+      <mass value="1.2" />
+      <inertia ixx="0.002" ixy="0.0" ixz="0.0" iyy="0.002" iyz="0.0" izz="0.002" />
     </inertial>
     <visual>
@@ -133,51 +152,29 @@
     </visual>
     <collision>
-      <origin xyz="0.16 0 0" rpy="0 0 0" />
-      <geometry>
-        <box size="0.22 0.022 0.022"/>
-      </geometry>
-    </collision>
-  </link>
-  <joint name="tibia_joint_FL" type="revolute">
-    <origin xyz="0.164 0 0" rpy="0 0 0" />
-    <parent link="femur_FL" />
-    <child link="tibia_FL" />
-    <axis xyz="0 0 -1" />
-    <dynamics damping="0.2" friction="0.02" />
-    <limit lower="-2.4" upper="2.4" effort="60" velocity="16"/>
-  </joint>
-  <joint name="foot_fixed_FL" type="fixed" dont_collapse="true">
-    <origin xyz="0.31 0 0" rpy="0 0 0" />
-    <parent link="tibia_FL" />
-    <child link="foot_FL" />
-  </joint>
-  <link name="foot_FL">
-    <inertial>
-      <origin xyz="0 0 0" rpy="0 0 0" />
-      <mass value="0.03" />
-      <inertia ixx="4.0e-6" ixy="0.0" ixz="0.0" iyy="4.0e-6" iyz="0.0" izz="4.0e-6" />
-    </inertial>
-    <visual>
-      <origin xyz="0 0 0" rpy="0 0 0" />
-      <geometry>
-        <sphere radius="0.01"/>
-      </geometry>
-      <material name="">
-        <color rgba="0.1 0.1 0.1 1" />
-      </material>
-    </visual>
-    <collision>
-      <origin xyz="0 0 0" rpy="0 0 0" />
-      <geometry>
-        <sphere radius="0.016"/>
-      </geometry>
-    </collision>
-  </link>
-  <!-- ==================== RL Leg ==================== -->
+      <origin xyz="0.29 0 -0.01" rpy="0 0 0" />
+      <geometry>
+        <sphere radius="0.02" />
+      </geometry>
+    </collision>
+  </link>
+  <joint
+    name="tibia_joint_FL"
+    type="continuous">
+    <origin
+      xyz="0.164 0 0"
+      rpy="0 0 0" />
+    <parent
+      link="femur_FL" />
+    <child
+      link="tibia_FL" />
+    <axis
+      xyz="0 0 -1" />
+    <limit effort="50" velocity="2"/>
+  </joint>
   <link name="coxa_RL">
     <inertial>
       <origin xyz="0.04 0 0" rpy="0 0 0" />
-      <mass value="0.08" />
-      <inertia ixx="1.5e-5" ixy="0.0" ixz="0.0" iyy="5.0e-5" iyz="0.0" izz="5.0e-5" />
+      <mass value="0.15" />
+      <inertia ixx="0.0001" ixy="0.0" ixz="0.0" iyy="0.0001" iyz="0.0" izz="0.0001" />
     </inertial>
     <visual>
@@ -197,17 +194,23 @@
     </collision>
   </link>
-  <joint name="coxa_joint_RL" type="revolute">
-    <origin xyz="-0.10275 0.11525 0" rpy="0 0 0" />
-    <parent link="base_link" />
-    <child link="coxa_RL" />
-    <axis xyz="0 0 1" />
-    <dynamics damping="0.2" friction="0.02" />
-    <limit lower="-0.9" upper="0.9" effort="60" velocity="12"/>
+  <joint
+    name="coxa_joint_RL"
+    type="continuous">
+    <origin
+      xyz="-0.10275 0.11525 0"
+      rpy="0 0 0" />
+    <parent
+      link="base_link" />
+    <child
+      link="coxa_RL" />
+    <axis
+      xyz="0 0 1" />
+    <limit effort="50" velocity="2"/>
   </joint>
   <link name="femur_RL">
     <inertial>
       <origin xyz="0.08 0 0" rpy="0 0 0" />
-      <mass value="0.32" />
-      <inertia ixx="8.0e-5" ixy="0.0" ixz="0.0" iyy="7.5e-4" iyz="0.0" izz="7.5e-4" />
+      <mass value="1.5" />
+      <inertia ixx="0.003" ixy="0.0" ixz="0.0" iyy="0.003" iyz="0.0" izz="0.003" />
     </inertial>
     <visual>
@@ -221,23 +224,29 @@
     </visual>
     <collision>
-      <origin xyz="0.08 0 -0.015" rpy="0 0 0" />
-      <geometry>
-        <box size="0.14 0.03 0.03"/>
-      </geometry>
-    </collision>
-  </link>
-  <joint name="femur_joint_RL" type="revolute">
-    <origin xyz="-0.0635321928743236 0.0437332030011001 0.0255" rpy="-1.5707963267949 0 2.35619449019235" />
-    <parent link="coxa_RL" />
-    <child link="femur_RL" />
-    <axis xyz="0 0 -1" />
-    <dynamics damping="0.2" friction="0.02" />
-    <limit lower="-1.6" upper="1.6" effort="60" velocity="16"/>
+      <origin xyz="0.06 0 -0.02" rpy="0 0 0" />
+      <geometry>
+        <box size="0.12 0.04 0.04"/>
+      </geometry>
+    </collision>
+  </link>
+  <joint
+    name="femur_joint_RL"
+    type="continuous">
+    <origin
+      xyz="-0.0635321928743236 0.0437332030011001 0.0255"
+      rpy="-1.5707963267949 0 2.35619449019235" />
+    <parent
+      link="coxa_RL" />
+    <child
+      link="femur_RL" />
+    <axis
+      xyz="0 0 -1" />
+    <limit effort="50" velocity="2"/>
   </joint>
   <link name="tibia_RL">
     <inertial>
-      <origin xyz="0.16 0 0" rpy="0 0 0" />
-      <mass value="0.16" />
-      <inertia ixx="2.0e-5" ixy="0.0" ixz="0.0" iyy="8.0e-4" iyz="0.0" izz="8.0e-4" />
+      <origin xyz="0.18 0 0" rpy="0 0 0" />
+      <mass value="1.2" />
+      <inertia ixx="0.002" ixy="0.0" ixz="0.0" iyy="0.002" iyz="0.0" izz="0.002" />
     </inertial>
     <visual>
@@ -251,51 +260,29 @@
     </visual>
     <collision>
-      <origin xyz="0.16 0 0" rpy="0 0 0" />
-      <geometry>
-        <box size="0.22 0.022 0.022"/>
-      </geometry>
-    </collision>
-  </link>
-  <joint name="tibia_joint_RL" type="revolute">
-    <origin xyz="0.164 0 0" rpy="0 0 0" />
-    <parent link="femur_RL" />
-    <child link="tibia_RL" />
-    <axis xyz="0 0 -1" />
-    <dynamics damping="0.2" friction="0.02" />
-    <limit lower="-2.4" upper="2.4" effort="60" velocity="16"/>
-  </joint>
-  <joint name="foot_fixed_RL" type="fixed" dont_collapse="true">
-    <origin xyz="0.31 0 0" rpy="0 0 0" />
-    <parent link="tibia_RL" />
-    <child link="foot_RL" />
-  </joint>
-  <link name="foot_RL">
-    <inertial>
-      <origin xyz="0 0 0" rpy="0 0 0" />
-      <mass value="0.03" />
-      <inertia ixx="4.0e-6" ixy="0.0" ixz="0.0" iyy="4.0e-6" iyz="0.0" izz="4.0e-6" />
-    </inertial>
-    <visual>
-      <origin xyz="0 0 0" rpy="0 0 0" />
-      <geometry>
-        <sphere radius="0.01"/>
-      </geometry>
-      <material name="">
-        <color rgba="0.1 0.1 0.1 1" />
-      </material>
-    </visual>
-    <collision>
-      <origin xyz="0 0 0" rpy="0 0 0" />
-      <geometry>
-        <sphere radius="0.016"/>
-      </geometry>
-    </collision>
-  </link>
-  <!-- ==================== FR Leg ==================== -->
+      <origin xyz="0.29 0 -0.01" rpy="0 0 0" />
+      <geometry>
+        <sphere radius="0.02" />
+      </geometry>
+    </collision>
+  </link>
+  <joint
+    name="tibia_joint_RL"
+    type="continuous">
+    <origin
+      xyz="0.164 0 0"
+      rpy="0 0 0" />
+    <parent
+      link="femur_RL" />
+    <child
+      link="tibia_RL" />
+    <axis
+      xyz="0 0 -1" />
+    <limit effort="50" velocity="2"/>
+  </joint>
   <link name="coxa_FR">
     <inertial>
       <origin xyz="0.04 0 0" rpy="0 0 0" />
-      <mass value="0.08" />
-      <inertia ixx="1.5e-5" ixy="0.0" ixz="0.0" iyy="5.0e-5" iyz="0.0" izz="5.0e-5" />
+      <mass value="0.15" />
+      <inertia ixx="0.0001" ixy="0.0" ixz="0.0" iyy="0.0001" iyz="0.0" izz="0.0001" />
     </inertial>
     <visual>
@@ -315,17 +302,23 @@
     </collision>
   </link>
-  <joint name="coxa_joint_FR" type="revolute">
-    <origin xyz="0.10275 -0.11525 0" rpy="0 0 0" />
-    <parent link="base_link" />
-    <child link="coxa_FR" />
-    <axis xyz="0 0 1" />
-    <dynamics damping="0.2" friction="0.02" />
-    <limit lower="-0.9" upper="0.9" effort="60" velocity="12"/>
+  <joint
+    name="coxa_joint_FR"
+    type="continuous">
+    <origin
+      xyz="0.10275 -0.11525 0"
+      rpy="0 0 0" />
+    <parent
+      link="base_link" />
+    <child
+      link="coxa_FR" />
+    <axis
+      xyz="0 0 1" />
+    <limit effort="50" velocity="2"/>
   </joint>
   <link name="femur_FR">
     <inertial>
       <origin xyz="0.08 0 0" rpy="0 0 0" />
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